File: hardware/PoE-Speaker/RevE/KiCad-RevE/02_Bench_protection.kicad_sch (KiCad schematic)
At the start: 15 parts, among them Q3 PSMN4R8-100BSE, Q4 PSMN4R8-100BSE, U15 LTC4365HTS8#TRPBF

Commit message: docs: archive final engineered PCB handoffs
Parts:
- C120: Voltage rating 100 V -> (none)
