File: hardware/PoE-Speaker/RevE/KiCad-RevE/08_PoE_input_and_isolation.kicad_sch (KiCad schematic)
At the start: 21 parts, among them U1 Ag5800, U12 PC817X2NSZ9F, U13 PC817X2NSZ9F, U14 PC817X2NSZ9F

Commit message: docs: archive final engineered PCB handoffs
Parts:
- R3, R4, R5: Power Rating 0.25 -> (none)
