File: hardware/PoE-Speaker/RevE/KiCad-RevE/11_Shared_current_protection.kicad_sch (KiCad schematic)
At the start: 15 parts, among them U16 TPS26630RGER

Commit message: docs: archive final engineered PCB handoffs
Parts:
- C121, C123: Voltage rating 50 V -> (none)
- C122: Voltage rating 100 V -> (none)
