File: hardware/PoE-Speaker/RevE/KiCad-RevE/12_Speaker_amplifier_1.kicad_sch (KiCad schematic)
At the start: 21 parts, among them J3 MX2EDGR-5.08-02P-GN01-Cu-A

Commit message: docs: archive final engineered PCB handoffs
Parts:
- R15, R16: Power Rating 0.1 -> (none)
